File: CART-Breakout.sch (KiCad schematic (older format))
At the start: 9 parts, among them P1 CONN_01X05, P2 CONN_01X05, P3 CONN_01X05, P4 CONN_01X05, P5 CONN_01X05, P6 CONN_01X05

Commit message: Updated from KiCAD 4 to KiCAD 5.1.19
Parts:
- removed D1: YELLOW, LEDs:LED_1206, symbol Led_Small
- removed P1, P2, P3, P4, P5, P6: CONN_01X05, Pin_Headers:Pin_Header_Straight_1x05, symbol CONN_01X05
- removed R1: 1.5K, Resistors_SMD:R_1206_HandSoldering, symbol R_Small
- added D1: YELLOW, LED_SMD:LED_1206_3216Metric, symbol Device:LED_Small_ALT
- added L1: LOGO, Symbol:OSHW-Logo2_7.3x6mm_SilkScreen, symbol RetroBitLab:LOGO
- added L2: LOGO, Symbol:KiCad-Logo2_5mm_SilkScreen, symbol RetroBitLab:LOGO
- added P1, P2, P3, P4, P5, P6: Conn_01x05, Connector_PinHeader_2.54mm:PinHeader_1x05_P2.54mm_Vertical, symbol Connector_Generic:Conn_01x05
- added R1: 1.5K, Resistor_SMD:R_1206_3216Metric_Pad1.30x1.75mm_HandSolder, symbol Device:R_Small
- CART1: symbol ATARI-CARTRIDGE -> RetroBitLab:ATARI-CARTRIDGE
Connections:
- net labels added: A0, A1, A10, A11, A12, A2, A3, A4, A5, A6, A7, A8, A9, D0, D1, D2, D3, D4, D5, D6, D7, PHI2, RD4, RD5, R~W, ~CCTL, ~S4, ~S5
- wire segments 64 -> 66
